Commit message: Phase 2 (World): Warehouse environment + robot table mount fix
World (warehouse_gazebo):
- warehouse.sdf: 12x10m warehouse with concrete floor, yellow cell markings
- Walls on 3 sides (South open for camera view), windows on North + East walls
- Directional sun + 2 overhead point lights above workspace
- Robot mounting table (steel, 0.8x0.8x0.9m) at origin
- Pick table (wood, 1.2x0.6x0.75m) at y=1.55 with 6 coloured physics boxes (2x3 grid)
- Storage rack (2 shelves at z=0.55 and z=1.05) at x=-1.6
- Box size: 0.07x0.07x0.07m, mass: 0.2kg (fits Robotiq 2F-85 85mm opening)
- warehouse_modified.sdf: layout adjusted via Gazebo GUI (rack rotated/repositioned)
- warehouse.launch.py: spawns world + robot, GZ_SIM_RESOURCE_PATH set programmatically

Robot description (warehouse_description):
- Removed pedestal from ur5e_with_gripper.urdf.xacro
- Robot now mounts directly to world link, spawned at z=0.9 on robot table
- Cleaner TF tree: world -> base_link directly

Verified:
- All 3 controllers active in warehouse world
- Robot sitting correctly on table, no extra block
- Boxes have real physics, rack has collision geometry

File: warehouse_description/urdf/ur5e_with_gripper.urdf.xacro (robot description, xacro)
@@ -22,30 +22,9 @@
   <link name="world"/>
   <!-- ========== Pedestal ========== -->
-  <link name="pedestal">
-    <visual>
-      <origin xyz="0 0 0.25" rpy="0 0 0"/>
-      <geometry><box size="0.15 0.15 0.5"/></geometry>
-      <material name="grey"><color rgba="0.4 0.4 0.4 1.0"/></material>
-    </visual>
-    <collision>
-      <origin xyz="0 0 0.25" rpy="0 0 0"/>
-      <geometry><box size="0.15 0.15 0.5"/></geometry>
-    </collision>
-    <inertial>
-      <mass value="20.0"/>
-      <origin xyz="0 0 0.25"/>
-      <inertia ixx="0.4" ixy="0" ixz="0" iyy="0.4" iyz="0" izz="0.05"/>
-    </inertial>
-  </link>
-  <joint name="world_to_pedestal" type="fixed">
-    <parent link="world"/>
-    <child link="pedestal"/>
-    <origin xyz="0 0 0" rpy="0 0 0"/>
-  </joint>
   <!-- ========== UR5e arm (kinematics only) ========== -->
   <xacro:ur_robot
     name="$(arg name)"
     tf_prefix="$(arg tf_prefix)"
-    parent="pedestal"
+    parent="world"
     joint_limits_parameters_file="$(arg joint_limit_params)"
     kinematics_parameters_file="$(arg kinematics_params)"
@@ -56,5 +35,5 @@
     safety_k_position="$(arg safety_k_position)"
     force_abs_paths="true">
-    <origin xyz="0 0 0.5" rpy="0 0 0"/>
+    <origin xyz="0 0 0" rpy="0 0 0"/>
   </xacro:ur_robot>
   <!-- ========== UR5e ros2_control (sim hardware) ========== -->
