Commit message: Phase 2 (Camera): Intel RealSense D435 eye-in-hand integration
warehouse_description:
- Added camera.xacro using official realsense2_description D435 macro
- Real D435 mesh visible in RViz (use_mesh:=true)
- Gazebo RGBD sensor block attached to camera_link
- Camera mounted on tool0 offset: xyz=(-0.03, -0.06, 0.02) rpy=(0, 1.57, 1.57)
- Added realsense2_description dependency to package.xml

warehouse_gazebo:
- Added gz-sim-sensors-system plugin to warehouse_modified.sdf
- Added image_bridge node for RGB + depth image topics
- Added parameter_bridge for PointCloud2 + CameraInfo
- lazy:=false on bridges to force eager mode

File: warehouse_description/urdf/camera.xacro (robot description, xacro)
@@ -1,44 +1,18 @@
 <?xml version="1.0"?>
 <robot xmlns:xacro="http://wiki.ros.org/xacro">
-  <xacro:macro name="realsense_d435" params="prefix parent *origin">
-    <!-- ========== Camera housing link ========== -->
-    <link name="${prefix}camera_link">
-      <visual>
-        <origin xyz="0 0 0" rpy="0 0 0"/>
-        <geometry>
-          <box size="0.025 0.090 0.025"/>
-        </geometry>
-        <material name="camera_grey">
-          <color rgba="0.2 0.2 0.2 1.0"/>
-        </material>
-      </visual>
-      <collision>
-        <origin xyz="0 0 0" rpy="0 0 0"/>
-        <geometry>
-          <box size="0.025 0.090 0.025"/>
-        </geometry>
-      </collision>
-      <inertial>
-        <mass value="0.072"/>
-        <origin xyz="0 0 0"/>
-        <inertia ixx="0.003881243" ixy="0" ixz="0"
-                 iyy="0.000498940" iyz="0"
-                 izz="0.003879257"/>
-      </inertial>
-    </link>
-    <!-- Camera mounted on flange via fixed joint -->
-    <joint name="${prefix}camera_joint" type="fixed">
-      <parent link="${parent}"/>
-      <child link="${prefix}camera_link"/>
+  <!-- Intel RealSense D435 — eye-in-hand mount -->
+  <!-- Uses official realsense2_description macro for real mesh -->
+  <!-- Adds Gazebo RGBD sensor block on top -->
+  <xacro:include filename="$(find realsense2_description)/urdf/_d435.urdf.xacro"/>
+  <xacro:macro name="realsense_d435_gazebo" params="prefix parent *origin">
+    <!-- Real D435 visual/collision/TF via official macro -->
+    <xacro:sensor_d435
+      name="${prefix}camera"
+      parent="${parent}"
+      use_nominal_extrinsics="true"
+      use_mesh="true">
       <xacro:insert_block name="origin"/>
-    </joint>
-    <!-- Optical frame — Z forward, X right, Y down (ROS convention) -->
-    <link name="${prefix}camera_optical_frame"/>
-    <joint name="${prefix}camera_optical_joint" type="fixed">
-      <parent link="${prefix}camera_link"/>
-      <child link="${prefix}camera_optical_frame"/>
-      <origin xyz="0 0 0" rpy="${-pi/2} 0 ${-pi/2}"/>
-    </joint>
-    <!-- ========== Gazebo RGBD sensor ========== -->
+    </xacro:sensor_d435>
+    <!-- Gazebo RGBD sensor attached to camera_link -->
     <gazebo reference="${prefix}camera_link">
       <sensor name="rgbd_camera" type="rgbd_camera">

File: warehouse_description/urdf/ur5e_with_gripper.urdf.xacro (robot description, xacro)
@@ -19,4 +19,5 @@
   <xacro:include filename="$(find robotiq_description)/urdf/robotiq_2f_85_macro.urdf.xacro"/>
   <xacro:include filename="$(find robotiq_description)/urdf/ur_to_robotiq_adapter.urdf.xacro"/>
+  <xacro:include filename="$(find warehouse_description)/urdf/camera.xacro"/>
   <!-- ========== World link ========== -->
   <link name="world"/>
@@ -55,5 +56,12 @@
     <origin xyz="0 0 0" rpy="0 0 0"/>
   </xacro:robotiq_gripper>
-<!-- ========== Gazebo: switch to bullet for mimic joint support ========== -->
+  <!-- ========== Intel RealSense D435 — eye-in-hand ========== -->
+  <xacro:realsense_d435_gazebo
+    prefix="$(arg tf_prefix)"
+    parent="$(arg tf_prefix)tool0">
+    <!-- Mounted forward of tool0, angled 30deg down toward workspace -->
+    <origin xyz="0.0 -0.08 -0.01" rpy="0 -1.57 1.57"/>
+  </xacro:realsense_d435_gazebo>
+<!-- ========== Gazebo: switch to bullet for mimic joint support my laptop is weaker ========== -->
   <gazebo>
     <physics type="bullet">
